File: kicad/lighthouse_display/lighthouse_display.kicad_sch (KiCad schematic)
At the start: 30 parts, among them J1 Conn_01x12_Pin, U1 IS31FL3731-SA, U2 TPS61176RTER, U3 SHTC3

Commit message: renamed libs + added opt3004 to lib
Changed lines of the file:
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@@
 (kicad_sch
-	(version 20231120)
+	(version 20250114)
 	(generator "eeschema")
-	(generator_version "8.0")
+	(generator_version "9.0")
 	(paper "A4")
+	(text "AD: set I2C address"
+		(exclude_from_sim no)
+		(at 83.058 91.948 0)
+		(effects
+			(font
+				(size 1.27 1.27)
+			)
+		)
+	)
+	(text "4.7uH: LSXND6060YEL4R7NMG "
+		(exclude_from_sim no)
+		(at 101.092 119.634 0)
+		(effects
+			(font
+				(size 1.27 1.27)
+			)
+		)
+	)
+	(text "7 white LEDs in series @ 20 mA -> 3.25 V\nVOUT 7*3.25 V = 22.75 V, VFB = 1.5\nVOUT = (Rupper/Rlower + 1) * 1.5 V\nRlower = Rupper / (VOUT/VFB - 1) = 70k5 @ Rupper = 1M\nRLower = 68k"
+		(exclude_from_sim no)
+		(at 107.95 186.69 0)
+		(effects
+			(font
+				(size 1.27 1.27)
+			)
+			(justify left)
+		)
+	)
+	(text "+12.0V\n+5.0V\n+3.3V"
+		(exclude_from_sim no)
+		(at 32.004 36.83 0)
+		(effects
+			(font
+				(size 1.27 1.27)
+			)
+		)
+	)
 	(junction
 		(at 43.18 138.43)
@@
 		)
 	)
-	(text "AD: set I2C address"
-		(exclude_from_sim no)
-		(at 83.058 91.948 0)
-		(effects
-			(font
-				(size 1.27 1.27)
-			)
-		)
-	)
-	(text "4.7uH: LSXND6060YEL4R7NMG "
-		(exclude_from_sim no)
-		(at 101.092 119.634 0)
-		(effects
-			(font
-				(size 1.27 1.27)
-			)
-		)
-	)
-	(text "7 white LEDs in series @ 20 mA -> 3.25 V\nVOUT 7*3.25 V = 22.75 V, VFB = 1.5\nVOUT = (Rupper/Rlower + 1) * 1.5 V\nRlower = Rupper / (VOUT/VFB - 1) = 70k5 @ Rupper = 1M\nRLower = 68k"
-		(exclude_from_sim no)
-		(at 107.95 186.69 0)
-		(effects
-			(font
-				(size 1.27 1.27)
-			)
-			(justify left)
-		)
-	)
-	(text "+12.0V\n+5.0V\n+3.3V"
-		(exclude_from_sim no)
-		(at 32.004 36.83 0)
-		(effects
-			(font
-				(size 1.27 1.27)
-			)
-		)
-	)
 	(label "IS_REXT"
 		(at 91.44 71.12 0)
-		(fields_autoplaced yes)
 		(effects
 			(font
@@
 	(label "IS_FILT"
 		(at 90.17 66.04 0)
-		(fields_autoplaced yes)
 		(effects
 			(font
@@
 	(label "SDA"
 		(at 66.04 45.72 0)
-		(fields_autoplaced yes)
 		(effects
 			(font
@@
 	(label "TPS_SW"
 		(at 119.38 138.43 90)
-		(fields_autoplaced yes)
 		(effects
 			(font
@@
 	(label "IS_IN"
 		(at 90.17 63.5 0)
-		(fields_autoplaced yes)
 		(effects
 			(font
@@
 	(label "TPS_LDO"
 		(at 71.12 165.1 0)
-		(fields_autoplaced yes)
 		(effects
 			(font
@@
 	(label "TPS_VIN"
 		(at 76.2 142.24 0)
-		(fields_autoplaced yes)
 		(effects
 			(font
@@
 	(label "SCL"
 		(at 66.04 48.26 0)
-		(fields_autoplaced yes)
 		(effects
 			(font
@@
 	(label "TPS_COMP"
 		(at 58.42 160.02 0)
-		(fields_autoplaced yes)
 		(effects
 			(font
@@
 	(label "TPS_ISET"
 		(at 81.28 170.18 0)
-		(fields_autoplaced yes)
 		(effects
 			(font
@@
 	(label "TPS_MODE"
 		(at 48.26 154.94 0)
-		(fields_autoplaced yes)
 		(effects
 			(font
@@
 	(label "~{SDB}"
 		(at 66.04 55.88 0)
-		(fields_autoplaced yes)
 		(effects
 			(font
@@
 	(label "WHITE_PWM"
 		(at 64.77 152.4 0)
-		(fields_autoplaced yes)
 		(effects
 			(font
@@
 	(label "IS_VIN"
 		(at 97.79 30.48 0)
-		(fields_autoplaced yes)
 		(effects
 			(font
@@
 	(label "~{INTB}"
 		(at 66.04 58.42 0)
-		(fields_autoplaced yes)
 		(effects
 			(font
@@
 	(label "IS_AD"
 		(at 90.17 50.8 0)
-		(fields_autoplaced yes)
 		(effects
 			(font
@@
 	(label "TPS_FB"
 		(at 121.92 147.32 0)
-		(fields_autoplaced yes)
 		(effects
 			(font
@@
 		(at 220.98 22.86)
 		(size 57.15 116.84)
+		(exclude_from_sim no)
+		(in_bom yes)
+		(on_board yes)
+		(dnp no)
 		(fields_autoplaced yes)
 		(stroke
@@
 		)
 	)
+	(embedded_fonts no)
 )

Commit message: ordererd lighthouse display
Parts:
- added C10: 100nF, Capacitor_SMD:C_0603_1608Metric_Pad1.08x0.95mm_HandSolder, symbol Device:C
- added IC1: OPT3004DNPR, lighthouse:SON65P200X200X65-7N-D, symbol lighthouse:OPT3004DNPR
- R6, R7: now not fitted
Connections:
- net +3.3V: now also C10.1, IC1.1 (VDD), IC1.2 (ADDR)
- net GND: now also C10.2, IC1.3 (GND), IC1.7 (EP)
- net SCL: now also IC1.4 (SCL)
- net SDA: now also IC1.6 (SDA)
- net WHITE_PWM: now also J1.12 (Pin_12)
- net ~{INTB}: now also J1.11 (Pin_11)
- net ~{SDB}: now also J1.10 (Pin_10)
- no-connect marks 3 -> 1
Other:
- note added: "I2C-Addr IS..: 0x74 SHTC3: 0x70 OPT3004: 0x45 (Addr VCC)"
